Commit message: fix gripper bug in gazebo by adding mimic_joint_plugin

File: src/xarm_description/urdf/arm.xacro (robot description, xacro)
@@ -23,4 +23,20 @@
         </inertial>
     </xacro:macro>
+    <xacro:macro name="mimic_joint_plugin_gazebo" params="name_prefix parent_joint mimic_joint has_pid:=false multiplier:=1.0 offset:=0 sensitiveness:=0.0 max_effort:=1.0 robot_namespace:=''">
+    <gazebo>
+      <plugin name="${name_prefix}mimic_joint_plugin" filename="libroboticsgroup_gazebo_mimic_joint_plugin.so">
+        <joint>${parent_joint}</joint>
+        <mimicJoint>${mimic_joint}</mimicJoint>
+        <xacro:if value="${has_pid}">                     <!-- if set to true, PID parameters from "/gazebo_ros_control/pid_gains/${mimic_joint}" are loaded -->
+          <hasPID />
+        </xacro:if>
+        <multiplier>${multiplier}</multiplier>
+        <offset>${offset}</offset>
+        <sensitiveness>${sensitiveness}</sensitiveness>   <!-- if absolute difference between setpoint and process value is below this threshold, do nothing; 0.0 = disable [rad] -->
+        <maxEffort>${max_effort}</maxEffort>              <!-- only taken into account if has_pid:=true [Nm] -->
+        <robotNamespace>/arm</robotNamespace>
+      </plugin>
+    </gazebo>
+  </xacro:macro>
     <!-- ///////////////////////////////////////   BOTTOM JOINT   ////////////////////////////////////////// -->
     <joint name="bottom_joint" type="fixed">
@@ -228,4 +244,7 @@
         <mimic joint="gripper_right_joint1" multiplier="1" offset="0" />
     </joint>
+    <xacro:mimic_joint_plugin_gazebo name_prefix="gripper_right_joint2"
+        parent_joint="gripper_right_joint1" mimic_joint="gripper_right_joint2"
+        has_pid="false" multiplier="1.0" max_effort="10.0" />
     <!-- ///////////////////////////////////////   GRIPPER RIGHT LINK2   ////////////////////////////////////////// -->
     <link name="gripper_right_link2">
@@ -255,4 +274,7 @@
         <mimic joint="gripper_right_joint1" multiplier="1" offset="0" />
     </joint>
+    <xacro:mimic_joint_plugin_gazebo name_prefix="gripper_left_joint1"
+        parent_joint="gripper_right_joint1" mimic_joint="gripper_left_joint1"
+        has_pid="false" multiplier="1.0" max_effort="10.0" />
     <!-- ///////////////////////////////////////   GRIPPER LEFT LINK1   ////////////////////////////////////////// -->
     <link name="gripper_left_link1">
@@ -282,4 +304,7 @@
         <mimic joint="gripper_right_joint2" multiplier="-1" offset="0" />
     </joint>
+    <xacro:mimic_joint_plugin_gazebo name_prefix="gripper_left_joint2"
+        parent_joint="gripper_right_joint2" mimic_joint="gripper_left_joint2"
+        has_pid="false" multiplier="-1.0" max_effort="10.0" />
     <!-- ///////////////////////////////////////   GRIPPER LEFT LINK2   ////////////////////////////////////////// -->
     <link name="gripper_left_link2">
